File: 04-implementation/01-pcb/MCU/01-mcu.brd (EAGLE design)
At the start: 71.1 x 55.9 mm, 49 parts, among them IC1 PIC24FJ128GB204, J2 ARDUINO-CONN-8X2, J3 ARDUINO-CONN-8X2, J4 ARDUINO-CONN-8, J6 ARDUINO-CONN-6, J7 PICKIT-ICSP, U2 ICE40-HX1K-VQFP100, U3 SP0502BAHT-SOT23, U4 MCP1700-SOT89, U6 MCP1700-SOT89

Commit message: Add files to release PCB after successful board bring up.
Parts:
- R7, R9: value 220 -> 680
Changed lines of the file:
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@@
 <?xml version="1.0" encoding="utf-8"?>
 <!DOCTYPE eagle SYSTEM "eagle.dtd">
-<eagle version="8.7.1">
+<eagle version="9.0.0">
 <drawing>
 <settings>
@@
 <attribute name="VALUE" x="15.048" y="53.567" size="1.27" layer="27" rot="R270"/>
 </element>
-<element name="R7" library="rcl" library_urn="urn:adsk.eagle:library:334" package="R0805" package3d_urn="urn:adsk.eagle:package:23553/2" value="220" x="14.5" y="50.4" smashed="yes">
+<element name="R7" library="rcl" library_urn="urn:adsk.eagle:library:334" package="R0805" package3d_urn="urn:adsk.eagle:package:23553/2" value="680" x="14.5" y="50.4" smashed="yes">
 <attribute name="NAME" x="10.54" y="49.789" size="1.27" layer="25"/>
 <attribute name="VALUE" x="13.865" y="47.86" size="1.27" layer="27"/>
@@
 <attribute name="VALUE" x="67.926" y="23.398" size="1.27" layer="27" rot="R90"/>
 </element>
-<element name="R9" library="rcl" library_urn="urn:adsk.eagle:library:334" package="R0805" package3d_urn="urn:adsk.eagle:package:23553/2" value="220" x="64.5" y="27.8" smashed="yes">
+<element name="R9" library="rcl" library_urn="urn:adsk.eagle:library:334" package="R0805" package3d_urn="urn:adsk.eagle:package:23553/2" value="680" x="64.5" y="27.8" smashed="yes">
 <attribute name="NAME" x="64.665" y="28.87" size="1.27" layer="25"/>
 <attribute name="VALUE" x="63.865" y="25.26" size="1.27" layer="27"/>
