File: 04-implementation/01-pcb/MIDI Input Port/MIDI Input.sch (EAGLE design)
At the start: 38 parts, among them J1 SDS-50J, J2 SDS-50J, J3 SDS-50J, J4 SDS-50J, J5 SSW-107-02-S-D, U1 PC900V, U2 PC900V, U3 PC900V, U4 PC900V

Commit message: Add files for PCB releases.
Parts:
- J5: value SSW-107-02-S-D -> SSW-107-02-G-D; device con-samtec:SSW-107-02-S-D -> MIDI router parts:SSW-107-02-G-D
