File: 04-implementation/01-pcb/MIDI Output Port/MIDI Output.sch (EAGLE design)
At the start: 34 parts, among them IC1 741G32, IC2 741G32, IC3 741G32, IC4 741G32, J1 SSW-107-02-S-D, U1 SDS-50J, U2 SDS-50J, U3 SDS-50J, U4 SDS-50J

Commit message: Revise MIDI PCB's for mechanical spacing of ribbon connector.
Parts:
- removed C1, C3, C5, C7, C9: 100n, rcl:C-EUC0805
Connections:
- removed net N$10: C3.1, U2.P$6, U2.P$7
- removed net N$19: C5.1, U3.P$6, U3.P$7
- removed net N$27: C7.1, U4.P$6, U4.P$7
- removed net N$6: C1.1, U1.P$6, U1.P$7
- net +5V: no longer C9.1
- net GND: now also U1.P$6, U1.P$7, U2.P$6, U2.P$7, U3.P$6, U3.P$7, U4.P$6, U4.P$7; no longer C1.2, C3.2, C5.2, C7.2, C9.2

Commit message: Add files for PCB releases.
Parts:
- J1: value SSW-107-02-S-D -> SSW-107-02-G-D; device con-samtec:SSW-107-02-S-D -> MIDI router parts:SSW-107-02-G-D
