File: 04-implementation/01-pcb/MCU/eagle/01-mcu.brd (EAGLE design)
At the start: 71.1 x 55.9 mm, 49 parts, among them IC1 PIC24FJ128GB204, J2 ARDUINO-CONN-8X2, J3 ARDUINO-CONN-8X2, J4 ARDUINO-CONN-8, J6 ARDUINO-CONN-6, J7 PICKIT-ICSP, U2 ICE40-HX1K-VQFP100, U3 SP0502BAHT-SOT23, U4 MCP1700-SOT89, U6 MCP1700-SOT89

Commit message: Add files for PCB releases.
Changed lines of the file:
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@@
 <?xml version="1.0" encoding="utf-8"?>
 <!DOCTYPE eagle SYSTEM "eagle.dtd">
-<eagle version="9.0.0">
+<eagle version="9.3.0">
 <drawing>
 <settings>
@@
 <setting verticaltext="up"/>
 </settings>
-<grid distance="0.1" unitdist="mm" unit="mm" style="lines" multiple="1" display="yes" altdistance="5" altunitdist="mil" altunit="mil"/>
+<grid distance="0.0999999999" unitdist="mm" unit="mm" style="lines" multiple="1" display="yes" altdistance="5" altunitdist="mil" altunit="mil"/>
 <layers>
 <layer number="1" name="Top" color="4" fill="1" visible="yes" active="yes"/>
@@
 <param name="checkStop" value="0"/>
 <param name="checkValues" value="0"/>
+<param name="checkNames" value="1"/>
+<param name="checkWireStubs" value="1"/>
+<param name="checkPolygonWidth" value="0"/>
 <param name="useDiameter" value="13"/>
 <param name="maxErrors" value="50"/>
@@
 </autorouter>
 <elements>
-<element name="C1" library="rcl" library_urn="urn:adsk.eagle:library:334" package="C0805" package3d_urn="urn:adsk.eagle:package:23617/2" value="100n" x="42.4" y="36.2">
+<element name="C1" library="rcl" library_urn="urn:adsk.eagle:library:334" package="C0805" package3d_urn="urn:adsk.eagle:package:23617/2" value="100n" x="42.4" y="36.2" smashed="yes">
+<attribute name="NAME" x="41.13" y="37.47" size="1.27" layer="25"/>
 <attribute name="SPICEPREFIX" value="C" x="42.4" y="36.2" size="1.778" layer="27" display="off"/>
+<attribute name="VALUE" x="41.13" y="33.66" size="1.27" layer="27"/>
 </element>
 <element name="C3" library="rcl" library_urn="urn:adsk.eagle:library:334" package="C0805" package3d_urn="urn:adsk.eagle:package:23617/2" value="100n" x="68.372" y="26.835" smashed="yes" rot="R90">
@@
 <attribute name="VALUE" x="29.54" y="19.92" size="1.778" layer="27" ratio="10" rot="R90"/>
 </element>
-<element name="L2" library="MIDI router MCU parts" package="L0805" value="BEAD" x="50.103" y="9.76"/>
+<element name="L2" library="MIDI router MCU parts" package="L0805" value="BEAD" x="50.103" y="9.76" smashed="yes">
+<attribute name="NAME" x="48.833" y="11.03" size="1.27" layer="25"/>
+<attribute name="VALUE" x="48.833" y="7.22" size="1.27" layer="27"/>
+</element>
 <element name="C17" library="rcl" library_urn="urn:adsk.eagle:library:334" package="C0805" package3d_urn="urn:adsk.eagle:package:23617/2" value="1u" x="4.6" y="41" smashed="yes">
 <attribute name="NAME" x="9.68" y="41.889" size="1.27" layer="25" rot="R180"/>
@@
 <attribute name="VALUE" x="66.331" y="23.897" size="1.27" layer="27" rot="R270"/>
 </element>
-<element name="IC1" library="MIDI router MCU parts" package="TQFP44" value="PIC24FJ128GB204" x="54.3" y="23.8"/>
+<element name="IC1" library="MIDI router MCU parts" package="TQFP44" value="PIC24FJ128GB204" x="54.3" y="23.8" smashed="yes">
+<attribute name="NAME" x="50.236" y="30.658" size="1.778" layer="25"/>
+<attribute name="VALUE" x="50.236" y="22.0299" size="1.778" layer="27"/>
+</element>
 <element name="R8" library="rcl" library_urn="urn:adsk.eagle:library:334" package="R0805" package3d_urn="urn:adsk.eagle:package:23553/2" value="10" x="43.7" y="19.8" smashed="yes">
 <attribute name="NAME" x="41.965" y="20.77" size="1.27" layer="25"/>
@@
 </signal>
 </signals>
+<mfgpreviewcolors>
+<mfgpreviewcolor name="soldermaskcolor" color="0xC8008000"/>
+<mfgpreviewcolor name="silkscreencolor" color="0xFFFEFEFE"/>
+<mfgpreviewcolor name="backgroundcolor" color="0xFF282828"/>
+<mfgpreviewcolor name="coppercolor" color="0xFFFFBF00"/>
+<mfgpreviewcolor name="substratecolor" color="0xFF786E46"/>
+</mfgpreviewcolors>
 </board>
 </drawing>

Commit message: Add files for pushbutton PCB.
Parts:
- U4, U6: device MIDI router MCU parts:MCP1700-SOT89 -> MIDI router parts:MCP1700-SOT89
Routing:
- net GND: track 107.3 -> 108.5 mm
- net VCCINT: track 13.7 -> 14.4 mm
- net +5V: vias 3 -> 10
