File: 04-implementation/01-pcb/MCU/eagle/01-mcu.sch (EAGLE design)
At the start: 49 parts, among them IC1 PIC24FJ128GB204, J2 ARDUINO-CONN-8X2, J3 ARDUINO-CONN-8X2, J4 ARDUINO-CONN-8, J6 ARDUINO-CONN-6, J7 PICKIT-ICSP, U2 ICE40-HX1K-VQFP100, U3 SP0502BAHT-SOT23, U4 MCP1700-SOT89, U6 MCP1700-SOT89

Commit message: Add files for pushbutton PCB.
Parts:
- U4, U6: device MIDI router MCU parts:MCP1700-SOT89 -> MIDI router parts:MCP1700-SOT89
